File: KiCad/DuoDiskAdapter.sch (KiCad schematic (older format))
At the start: 12 parts, among them J1 Apple II, J2 DuoDisk, J3 FloppyEmu, SW1 DRIVE1, SW2 DRIVE2, SW3 SWAP 1/2

Commit message: Updated PCB and Gerber files.
Other:
- note added: "SW1 connects DRIVE1 to DUODISK or FLOPPYEMU\nSW2 connects DRIVE2 to DUODISK or FLOPPYEMU\nSW3 swaps FLOPPYEMU's DRIVE1/DRIVE2"
- note removed: "SW1 connects DRIVE1 to A or B\nSW2 connects DRIVE2 to A or B\nSW3 swaps B's DRIVE1/DRIVE2"
- moved on the sheet: TP1
Changed lines of the file:
@@
 Rev "1.0"
 Comp "Thorsten Brehm"
-Comment1 ""
-Comment2 ""
+Comment1 "CC-BY-SA 4.0"
+Comment2 "FloppyEmu-DuoDisk-Adapter for the Apple II"
 Comment3 ""
 Comment4 ""
@@
 GND2
 Text Notes 5100 4300 0    50   ~ 0
-SW1 connects DRIVE1 to A or B\nSW2 connects DRIVE2 to A or B\nSW3 swaps B's DRIVE1/DRIVE2
+SW1 connects DRIVE1 to DUODISK or FLOPPYEMU\nSW2 connects DRIVE2 to DUODISK or FLOPPYEMU\nSW3 swaps FLOPPYEMU's DRIVE1/DRIVE2
 Wire Notes Line
 	5050 1150 5050 4350
@@
 Wire Wire Line
 	2150 4200 2300 4200
-Text GLabel 6500 4600 0    50   Input ~ 0
+Text GLabel 6000 4700 0    50   Input ~ 0
 GND
 $Comp
 L Connector:TestPoint TP1
 U 1 1 62B6B05E
-P 6800 4600
-F 0 "TP1" V 6754 4788 50  0000 L CNN
-F 1 "GND" V 6845 4788 50  0000 L CNN
-F 2 "Measurement_Points:Measurement_Point_Round-TH_Small" H 7000 4600 50  0001 C CNN
-F 3 "~" H 7000 4600 50  0001 C CNN
-	1    6800 4600
+P 6300 4700
+F 0 "TP1" V 6254 4888 50  0000 L CNN
+F 1 "GND" V 6345 4888 50  0000 L CNN
+F 2 "Measurement_Points:Measurement_Point_Round-TH_Small" H 6500 4700 50  0001 C CNN
+F 3 "~" H 6500 4700 50  0001 C CNN
+	1    6300 4700
 	0    1    1    0
 $EndComp
 Wire Wire Line
-	6800 4600 6500 4600
+	6300 4700 6000 4700
 Wire Notes Line
 	5050 4450 7850 4450
@@
 Wire Wire Line
 	1850 4650 2350 4650
-Wire Notes Line
-	850  1150 4600 1150
 Wire Wire Line
 	1550 2250 2100 2250
@@
 Wire Wire Line
 	3400 1950 3400 1700
+Wire Notes Line
+	850  1150 4900 1150
 $EndSCHEMATC

Commit message: v1.1: fixed FloppyEmu connector: Added extra +5V connection to pin 11.
Connections:
- net _+5V: now also J3.11 (Pin_11)
- no-connect marks 14 -> 13
Changed lines of the file:
@@
 Sheet 1 1
 Title "DuoDisk-FloppyEmu Adapter"
-Date "2022-06-05"
-Rev "1.0"
+Date "2022-06-21"
+Rev "1.1"
 Comp "Thorsten Brehm"
 Comment1 "CC-BY-SA 4.0"
@@
 	2100 4750 2100 2250
 NoConn ~ 2350 4850
-NoConn ~ 2350 4950
 NoConn ~ 2350 5050
 NoConn ~ 2350 5150
@@
 	1550 2750 4300 2750
 Wire Wire Line
-	1550 2850 4300 2850
+	1550 2850 2050 2850
 Wire Wire Line
 	1550 2950 4300 2950
@@
 Wire Notes Line
 	850  1150 4900 1150
+Wire Wire Line
+	2350 4950 2050 4950
+Wire Wire Line
+	2050 4950 2050 2850
+Connection ~ 2050 2850
+Wire Wire Line
+	2050 2850 4300 2850
+Text Label 2100 4950 0    50   ~ 0
+_+5V
 $EndSCHEMATC

Commit message: Changed pull-ups to 10K. 10K is enough and reduces load (especially since the disk drive itself usually also has a pull-up).
Parts:
- R2, R3, R4, R5: value 3K3 -> 10K
Changed lines of the file:
@@
 P 5950 2700
 F 0 "R2" H 6100 2650 50  0000 R CNN
-F 1 "3K3" H 6150 2750 50  0000 R CNN
+F 1 "10K" H 6150 2750 50  0000 R CNN
 F 2 "Resistors_THT:R_Axial_DIN0207_L6.3mm_D2.5mm_P10.16mm_Horizontal" V 5880 2700 50  0001 C CNN
 F 3 "~" H 5950 2700 50  0001 C CNN
@@
 P 7100 3000
 F 0 "R3" H 7170 3046 50  0000 L CNN
-F 1 "3K3" H 7170 2955 50  0000 L CNN
+F 1 "10K" H 7170 2955 50  0000 L CNN
 F 2 "Resistors_THT:R_Axial_DIN0207_L6.3mm_D2.5mm_P10.16mm_Horizontal" V 7030 3000 50  0001 C CNN
 F 3 "~" H 7100 3000 50  0001 C CNN
@@
 P 7100 2700
 F 0 "R4" H 6950 2750 50  0000 L CNN
-F 1 "3K3" H 6900 2650 50  0000 L CNN
+F 1 "10K" H 6900 2650 50  0000 L CNN
 F 2 "Resistors_THT:R_Axial_DIN0207_L6.3mm_D2.5mm_P10.16mm_Horizontal" V 7030 2700 50  0001 C CNN
 F 3 "~" H 7100 2700 50  0001 C CNN
@@
 P 6800 3000
 F 0 "R5" H 6870 3046 50  0000 L CNN
-F 1 "3K3" H 6870 2955 50  0000 L CNN
+F 1 "10K" H 6870 2955 50  0000 L CNN
 F 2 "Resistors_THT:R_Axial_DIN0207_L6.3mm_D2.5mm_P10.16mm_Horizontal" V 6730 3000 50  0001 C CNN
 F 3 "~" H 6800 3000 50  0001 C CNN

Commit message: Updated KiCad design files to reflect correct pin name for D-SUB/pin21. D-SUB/pin 21 is actually not a ground pin, but the "/Apple II emulation" pin. It is just hard-wired to GND by the AppleII cables - since it wants the DuoDisk to always operate in AppleII mode. (This disables the disk-swap-detect logic, which the Disk III introduced - and which the DuoDisk indeed also has, though the Apple IIs keep it disabled).
Connections:
- net GND4 renamed ~A2Emulation
Changed lines of the file:
@@
 GND3
 Text Label 1650 2550 0    50   ~ 0
-GND4
+~A2Emulation
 Connection ~ 2150 4200
 Wire Wire Line
