File: KiCad/DuoDiskAdapter.kicad_pcb (KiCad board)
At the start: 2 copper layers, 59.4 x 46.3 mm, 13 parts, among them J1 Apple II, J2 DuoDisk, J3 FloppyEmu, SW1 DRIVE1, SW2 DRIVE2, SW3 SWAP 1/2

Commit message: Updated PCB and Gerber files.
Parts:
- removed the REF*** at (129.3, 77.8)
- added REF***: OSHW-Logo2_9.8x8mm_SilkScreen, Symbols:OSHW-Logo2_9.8x8mm_SilkScreen, F.Cu at (128.9, 75.1)
- moved J3 5.47 mm to (101.5, 74.6)
- moved J1 2.00 mm to (79.7, 58.7)
- moved SW1 1.00 mm to (108.9, 83.7)
- moved SW2 1.00 mm to (121.9, 83.7)
- moved SW3 1.00 mm to (83.0, 72.7)
Routing:
- net ~FE_ENABLE2: track 40.6 -> 54.4 mm
- net GND: track 125.2 -> 131.9 mm
- net /+12V: track 78.8 -> 84.0 mm
- net /~FE_ENABLE1_SW: track 26.5 -> 21.5 mm
- net +5V: track 118.6 -> 121.5 mm
- net /PHASE3: track 59.0 -> 61.7 mm
- net /_+5V: track 84.2 -> 86.8 mm
- net /PHASE1: track 59.5 -> 62.1 mm
- net /PHASE2: track 59.2 -> 61.6 mm
- net /-12V: track 64.1 -> 66.5 mm
- net /WREQ: track 61.8 -> 64.2 mm
- net /GND4: track 79.1 -> 81.4 mm
- net /WR: track 68.1 -> 70.3 mm
- net /GND3: track 56.0 -> 58.2 mm
- net /RD: track 80.1 -> 82.1 mm
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Other:
- board size 59.4 x 46.3 mm -> 61.4 x 46.3 mm
- board text added: "APPLE ÜÄ :)"
- board text added: "Apple II DuoDisk FloppyEmu Adapter v1.0"
- board text added: "CC-BY-SA 4.0"
- board text added: "FloppyEmu"
- board text removed: "Apple II DuoDisk FloppyEmu Adapter"

Commit message: v1.1: fixed FloppyEmu connector: Added extra +5V connection to pin 11.
Connections:
- J3 pad 11: Net-(J3-Pad11) -> /_+5V
Routing:
- net /_+5V: track 86.8 -> 106.9 mm
- net ~FE_ENABLE1: track 49.3 -> 51.1 mm
- net /RD: track 82.1 -> 81.6 mm
Other:
- board text added: "Apple II DuoDisk FloppyEmu Adapter v1.1"
- board text removed: "Apple II DuoDisk FloppyEmu Adapter v1.0"

Commit message: Changed pull-ups to 10K. 10K is enough and reduces load (especially since the disk drive itself usually also has a pull-up).
Parts:
- R2, R3, R4, R5: value 3K3 -> 10K

Commit message: Updated KiCad design files to reflect correct pin name for D-SUB/pin21. D-SUB/pin 21 is actually not a ground pin, but the "/Apple II emulation" pin. It is just hard-wired to GND by the AppleII cables - since it wants the DuoDisk to always operate in AppleII mode. (This disables the disk-swap-detect logic, which the Disk III introduced - and which the DuoDisk indeed also has, though the Apple IIs keep it disabled).
Connections:
- net /GND4 renamed /~A2Emulation
Changed lines of the file:
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@@
   (net 30 /GND1)
   (net 31 /_+5V)
-  (net 32 /GND4)
+  (net 32 /~A2Emulation)
   (net 33 /GND3)
   (net 34 GND)
@@
     (add_net /GND2)
     (add_net /GND3)
-    (add_net /GND4)
+    (add_net /~A2Emulation)
     (add_net /PHASE0)
     (add_net /PHASE1)
@@
       (net 5 /+12V))
     (pad 21 smd rect (at -4.155 0 270) (size 1.846667 3.48) (layers B.Cu B.Paste B.Mask)
-      (net 32 /GND4))
+      (net 32 /~A2Emulation))
     (pad 22 smd rect (at -6.925 0 270) (size 1.846667 3.48) (layers B.Cu B.Paste B.Mask)
       (net 4 "Net-(J1-Pad22)"))
@@
       (net 17 "Net-(J2-Pad22)"))
     (pad 21 smd rect (at 4.155 0 90) (size 1.846667 3.48) (layers B.Cu B.Paste B.Mask)
-      (net 32 /GND4))
+      (net 32 /~A2Emulation))
     (pad 20 smd rect (at 1.385 0 90) (size 1.846667 3.48) (layers B.Cu B.Paste B.Mask)
       (net 5 /+12V))

Commit message: v2.0: added solder jumpers for +/-12V These are not required for FloppyEmu (should be left open). Closing the jumpers provides the option to connect real Disk II drives.
Parts:
- added JP1: -12V, Jumper:SolderJumper-2_P1.3mm_Open_RoundedPad1.0x1.5mm, F.Cu at (116.6, 50.5)
- added JP2: +12V, Jumper:SolderJumper-2_P1.3mm_Open_RoundedPad1.0x1.5mm, B.Cu at (87.0, 59.3)
Connections:
- net /~A2Emulation renamed /~{A2Emulation}
- net /~FE_ENABLE1_SW renamed /~{FE_ENABLE1_SW}
- net /~FE_ENABLE2_R renamed /~{FE_ENABLE2_R}
- net /~FE_ENABLE2_SW renamed /~{FE_ENABLE2_SW}
- net ~DUO_ENABLE1 renamed ~{DUO_ENABLE1}
- net ~DUO_ENABLE2 renamed ~{DUO_ENABLE2}
- net ~ENABLE1 renamed ~{ENABLE1}
- net ~ENABLE2 renamed ~{ENABLE2}
- net ~FE_ENABLE1 renamed ~{FE_ENABLE1}
- net ~FE_ENABLE2 renamed ~{FE_ENABLE2}
- J1 pad 1: Net-(J1-Pad1) -> unconnected-(J1-Pad1)
- J1 pad 13: Net-(J1-Pad13) -> unconnected-(J1-Pad13)
- J1 pad 22: Net-(J1-Pad22) -> unconnected-(J1-Pad22)
- J1 pad 25: Net-(J1-Pad25) -> unconnected-(J1-Pad25)
- J2 pad 1: Net-(J2-Pad1) -> unconnected-(J2-Pad1)
- J2 pad 13: Net-(J2-Pad13) -> unconnected-(J2-Pad13)
- J2 pad 22: Net-(J2-Pad22) -> unconnected-(J2-Pad22)
- J2 pad 25: Net-(J2-Pad25) -> unconnected-(J2-Pad25)
- J3 pad 13: Net-(J3-Pad13) -> Net-(J3-Pad17)
- J3 pad 15: Net-(J3-Pad15) -> Net-(J3-Pad17)
- J3 pad 19: Net-(J3-Pad19) -> Net-(J3-Pad17)
Routing:
- net Net-(J3-Pad17): track 0.00 -> 36.6 mm
- net Net-(J3-Pad9): track 0.00 -> 18.1 mm
- net /-12V: track 66.5 -> 74.9 mm, vias 0 -> 1
- net /GND2: track 91.4 -> 85.4 mm
- net GND: track 131.9 -> 127.5 mm
- net /_+5V: track 106.9 -> 102.7 mm
- net /PHASE2: track 61.6 -> 59.8 mm
- net ~{DUO_ENABLE1}: track 55.3 -> 53.6 mm
- net ~{ENABLE2}: track 58.4 -> 57.0 mm
- net /+12V: track 84.0 -> 85.3 mm
- net /PHASE0: track 61.8 -> 60.6 mm
- net /PHASE1: track 62.1 -> 61.0 mm
- net /PHASE3: track 61.7 -> 60.8 mm
- net /~{FE_ENABLE2_SW}: track 43.7 -> 42.7 mm
- net /GND1: track 73.3 -> 72.4 mm
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Other:
- net class Default removed
- board text added: "Apple II DuoDisk FloppyEmu Adapter v2.0"
- board text removed: "Apple II DuoDisk FloppyEmu Adapter v1.1"
